Commit message: Lidar and Depth Camera implementation

File: g1_description/urdf/g1_29dof.urdf (robot description, URDF)
Before this commit: robot g1_29dof, 40 links, 39 joints
Links:
- added link d435_link_optical
Joints:
- added joint d435_optical_joint: type fixed, parent d435_link, child d435_link_optical, origin xyz=0 0 0 rpy=-1.5708 0 -1.5708
