Commit message: Feat: Project conclusion

File: src/g1_description/urdf/g1_29dof_2d.urdf (robot description, URDF)
Before this commit: robot g1_29dof, 42 links, 41 joints
Joints:
- joint left_elbow_joint: origin xyz=0.015783 0 -0.080518 rpy=0 0 0 -> xyz=0.015783 0 -0.080518 rpy=0 1.2 0
- joint left_shoulder_pitch_joint: origin xyz=0.0039563 0.10022 0.23778 rpy=0.27931 5.4949E-05 -0.00019159 -> xyz=0.0039563 0.10022 0.23778 rpy=0 0 0
- joint left_shoulder_roll_joint: origin xyz=0 0.038 -0.013831 rpy=-0.27925 0 0 -> xyz=0 0.038 -0.013831 rpy=0 0 0
- joint right_elbow_joint: origin xyz=0.015783 0 -0.080518 rpy=0 0 0 -> xyz=0.015783 0 -0.080518 rpy=0 1.2 0
- joint right_shoulder_pitch_joint: origin xyz=0.0039563 -0.10021 0.23778 rpy=-0.27931 5.4949E-05 0.00019159 -> xyz=0.0039563 -0.10021 0.23778 rpy=0 0 0
- joint right_shoulder_roll_joint: origin xyz=0 -0.038 -0.013831 rpy=0.27925 0 0 -> xyz=0 -0.038 -0.013831 rpy=0 0 0

File: src/g1_description/urdf/g1_29dof_3d.urdf (robot description, URDF)
Before this commit: robot g1_29dof, 43 links, 42 joints
Joints:
- joint left_ankle_pitch_joint: axis 0 1 0 -> (none); limit lower=-0.87267 upper=0.5236 effort=35 velocity=30 -> (none); type revolute -> fixed
- joint left_ankle_roll_joint: axis 1 0 0 -> (none); limit lower=-0.2618 upper=0.2618 effort=35 velocity=30 -> (none); type revolute -> fixed
- joint left_elbow_joint: axis 0 1 0 -> (none); limit lower=-1.0472 upper=2.0944 effort=25 velocity=37 -> (none); origin xyz=0.015783 0 -0.080518 rpy=0 0 0 -> xyz=0.015783 0 -0.080518 rpy=0 1.2 0; type revolute -> fixed
- joint left_hip_pitch_joint: axis 0 1 0 -> (none); limit lower=-2.5307 upper=2.8798 effort=88 velocity=32 -> (none); type revolute -> fixed
- joint left_hip_roll_joint: axis 1 0 0 -> (none); limit lower=-0.5236 upper=2.9671 effort=88 velocity=32 -> (none); type revolute -> fixed
- joint left_hip_yaw_joint: axis 0 0 1 -> (none); limit lower=-2.7576 upper=2.7576 effort=88 velocity=32 -> (none); type revolute -> fixed
- joint left_knee_joint: axis 0 1 0 -> (none); limit lower=-0.087267 upper=2.8798 effort=139 velocity=20 -> (none); type revolute -> fixed
- joint left_shoulder_pitch_joint: axis 0 1 0 -> (none); limit lower=-3.0892 upper=2.6704 effort=25 velocity=37 -> (none); origin xyz=0.0039563 0.10022 0.23778 rpy=0.27931 1.5708 -0.00019159 -> xyz=0.0039563 0.10022 0.23778 rpy=0 0 0; type revolute -> fixed
- joint left_shoulder_roll_joint: axis 1 0 0 -> (none); limit lower=-1.5882 upper=2.2515 effort=25 velocity=37 -> (none); origin xyz=0 0.038 -0.013831 rpy=-0.27925 0 0 -> xyz=0 0.038 -0.013831 rpy=0 0 0; type revolute -> fixed
- joint left_shoulder_yaw_joint: axis 0 0 1 -> (none); limit lower=-2.618 upper=2.618 effort=25 velocity=37 -> (none); type revolute -> fixed
- joint left_wrist_pitch_joint: axis 0 1 0 -> (none); limit lower=-1.61 upper=1.61 effort=5 velocity=22 -> (none); type revolute -> fixed
- joint left_wrist_roll_joint: axis 1 0 0 -> (none); limit lower=-1.97 upper=1.97 effort=25 velocity=37 -> (none); type revolute -> fixed
- joint left_wrist_yaw_joint: axis 0 0 1 -> (none); limit lower=-1.61 upper=1.61 effort=5 velocity=22 -> (none); type revolute -> fixed
- joint right_ankle_pitch_joint: axis 0 1 0 -> (none); limit lower=-0.87267 upper=0.5236 effort=35 velocity=30 -> (none); type revolute -> fixed
- joint right_ankle_roll_joint: axis 1 0 0 -> (none); limit lower=-0.2618 upper=0.2618 effort=35 velocity=30 -> (none); type revolute -> fixed
- joint right_elbow_joint: axis 0 1 0 -> (none); limit lower=-1.0472 upper=2.0944 effort=25 velocity=37 -> (none); origin xyz=0.015783 0 -0.080518 rpy=0 0 0 -> xyz=0.015783 0 -0.080518 rpy=0 1.2 0; type revolute -> fixed
- joint right_hip_pitch_joint: axis 0 1 0 -> (none); limit lower=-2.5307 upper=2.8798 effort=88 velocity=32 -> (none); type revolute -> fixed
- joint right_hip_roll_joint: axis 1 0 0 -> (none); limit lower=-2.9671 upper=0.5236 effort=88 velocity=32 -> (none); type revolute -> fixed
- joint right_hip_yaw_joint: axis 0 0 1 -> (none); limit lower=-2.7576 upper=2.7576 effort=88 velocity=32 -> (none); type revolute -> fixed
- joint right_knee_joint: axis 0 1 0 -> (none); limit lower=-0.087267 upper=2.8798 effort=139 velocity=20 -> (none); type revolute -> fixed
- joint right_shoulder_pitch_joint: axis 0 1 0 -> (none); limit lower=-3.0892 upper=2.6704 effort=25 velocity=37 -> (none); origin xyz=0.0039563 -0.10021 0.23778 rpy=-0.27931 1.5708 0.00019159 -> xyz=0.0039563 -0.10021 0.23778 rpy=0 0 0; type revolute -> fixed
- joint right_shoulder_roll_joint: axis 1 0 0 -> (none); limit lower=-2.2515 upper=1.5882 effort=25 velocity=37 -> (none); origin xyz=0 -0.038 -0.013831 rpy=0.27925 0 0 -> xyz=0 -0.038 -0.013831 rpy=0 0 0; type revolute -> fixed
- joint right_shoulder_yaw_joint: axis 0 0 1 -> (none); limit lower=-2.618 upper=2.618 effort=25 velocity=37 -> (none); type revolute -> fixed
- joint right_wrist_pitch_joint: axis 0 1 0 -> (none); limit lower=-1.61 upper=1.61 effort=5 velocity=22 -> (none); type revolute -> fixed
- joint right_wrist_roll_joint: axis 1 0 0 -> (none); limit lower=-1.97 upper=1.97 effort=25 velocity=37 -> (none); type revolute -> fixed
- joint right_wrist_yaw_joint: axis 0 0 1 -> (none); limit lower=-1.61 upper=1.61 effort=5 velocity=22 -> (none); type revolute -> fixed
- joint waist_pitch_joint: axis 0 1 0 -> (none); limit lower=-0.52 upper=0.52 effort=35 velocity=30 -> (none); type revolute -> fixed
- joint waist_roll_joint: axis 1 0 0 -> (none); limit lower=-0.52 upper=0.52 effort=35 velocity=30 -> (none); type revolute -> fixed
- joint waist_yaw_joint: axis 0 0 1 -> (none); limit lower=-2.618 upper=2.618 effort=88 velocity=32 -> (none); type revolute -> fixed
