Commit message: Fix: RTABMAP mapping fixed

File: src/g1_description/urdf/g1_29dof_3d.urdf (robot description, URDF)
Before this commit: robot g1_29dof, 43 links, 42 joints
Joints:
- joint mid360_joint: origin xyz=0.0002835 0.00003 0.40618 rpy=0 0.04014257279586953 0 -> xyz=0.0002835 0.00003 0.40618 rpy=3.14159 0.04014257279586953 0
